File: _autosave-ProjectKurinda_PCB.kicad_sch (KiCad schematic)
At the start: 19 parts, among them J1 Conn_01x02, Q2 Q_PMOS_GSD, U1 ESP32-C3_SUPERMINI_TH, U2 SHT40, U3 Water Sensor, U4 RV3028 RTC, U5 LIS2DW12 breakout

Commit message: New version v1.1 of sensor PCB with new sensor modules and extra features, and updated README file.
Changed lines of the file:
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@@
 	(text "Sensor will operate without any surface-mount components\nif jumpers 1 and 2 are shorted with solder joints."
 		(exclude_from_sim no)
-		(at 219.456 141.478 0)
+		(at 242.062 161.544 0)
 		(effects
 			(font
